Commit message: sensors part commit

File: body.urdf (robot description, URDF)
Before this commit: robot robot, 3 links, 2 joints
Links:
- removed link L_Leg
- removed link R_Leg
- added link LLeg, mass 1; collision box size=1 1 1; visual box size=1 1 1
- added link RLeg, mass 1; collision box size=1 1 1; visual box size=1 1 1
Joints:
- removed joint Torso_L_Leg
- removed joint Torso_R_Leg
- added joint Torso_LLeg: type fixed, parent Torso, child LLeg, origin xyz=-0.5 0 1.0 rpy=0 0 0, axis 0 1 0, limit lower=-3.14159 upper=3.14159 effort=0.0 velocity=0.0
- added joint Torso_RLeg: type fixed, parent Torso, child RLeg, origin xyz=0.5 0 1.0 rpy=0 0 0, axis 0 1 0, limit lower=-3.14159 upper=3.14159 effort=0.0 velocity=0.0

Commit message: sensors part commit

File: body.urdf (robot description, URDF)
Before this commit: robot robot, 3 links, 2 joints
Joints:
- joint Torso_LLeg: type fixed -> revolute
- joint Torso_RLeg: type fixed -> revolute

Commit message: master push after refactoring

File: body.urdf (robot description, URDF)
Before this commit: robot robot, 2 links, 1 joints
Links:
- removed link Leg
- added link BLeg, mass 1; collision box size=1 1 1; visual box size=1 1 1
- added link FLeg, mass 1; collision box size=1 1 1; visual box size=1 1 1
Joints:
- removed joint Torso_Leg
- added joint Torso_BLeg: type revolute, parent Torso, child BLeg, origin xyz=-0.5 0 1 rpy=0 0 0, axis 0 1 0, limit lower=-3.14159 upper=3.14159 effort=0.0 velocity=0.0
- added joint Torso_FLeg: type revolute, parent Torso, child FLeg, origin xyz=0.5 0 1 rpy=0 0 0, axis 0 1 0, limit lower=-3.14159 upper=3.14159 effort=0.0 velocity=0.0

Commit message: master push after refactoring

File: body.urdf (robot description, URDF)
Before this commit: robot robot, 3 links, 2 joints
Joints:
- joint Torso_BLeg: origin xyz=-0.5 0 1 rpy=0 0 0 -> xyz=-0.5 0 1.5 rpy=0 0 0
- joint Torso_FLeg: origin xyz=0.5 0 1 rpy=0 0 0 -> xyz=0.5 0 1.5 rpy=0 0 0
